Commit message: added rviz and colors

File: urdf/open_manipulator_x.urdf.xacro (robot description, xacro)
@@ -231,5 +231,5 @@
     </inertial>
   </link>
-  <!-- <joint name="end_effector_joint" type="fixed">
+  <joint name="end_effector_joint" type="fixed">
     <origin xyz="0.126 0.0 0.0" rpy="0 0 0"/>
     <parent link="link5"/>
@@ -252,5 +252,5 @@
     </inertial>
   </link>
-  <joint name="camera_joint" type="fixed">
+  <!-- <joint name="camera_joint" type="fixed">
     <axis xyz="0 1 0" />
     <origin xyz="0.070 0.032 0.052" rpy="0 0 0"/>
@@ -264,5 +264,5 @@
         <box size="0.01 0.01 0.01" />
       </geometry>
-      <material name="red"/>
+      <material name="grey"/>
     </visual>
     <inertial>
@@ -346,3 +346,27 @@
     </plugin>
   </gazebo>
+  <gazebo reference="link1">
+    <material>Gazebo/black</material>
+  </gazebo>
+  <gazebo reference="link2">
+    <material>Gazebo/black</material>
+  </gazebo>
+  <gazebo reference="link3">
+    <material>Gazebo/black</material>
+  </gazebo>
+  <gazebo reference="link4">
+    <material>Gazebo/black</material>
+  </gazebo>
+  <gazebo reference="link5">
+    <material>Gazebo/black</material>
+  </gazebo>
+  <gazebo reference="gripper_link">
+    <material>Gazebo/black</material>
+  </gazebo>
+  <gazebo reference="gripper_link_sub">
+    <material>Gazebo/black</material>
+  </gazebo>
+  <gazebo reference="end_effector_link">
+    <material>Gazebo/RedBright</material>
+  </gazebo>
 </robot>
